Commit message: traj ready for testing

File: description/urdf/modularbot.urdf (robot description, URDF)
Before this commit: robot ModularBot, 33 links, 32 joints
Links:
- added link J1_E_stator, mass 3.586681; collision mesh filename=package://concert_resources/models/modular/meshes/concert/s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 scale=0.001 0.001 0.001; visual mesh filename=package://concert_resources/models/modular/meshes/concert/c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 scale=0.001 0.001 0.001
- added link J2_E_stator, mass 3.6144181; collision mesh filename=package://concert_resources/models/modular/meshes/concert/s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 scale=0.001 0.001 0.001; visual mesh filename=package://concert_resources/models/modular/meshes/concert/c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 scale=0.001 0.001 0.001
- added link J3_E_stator, mass 3.2592751; collision mesh filename=package://concert_resources/models/modular/meshes/concert/s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 scale=0.001 0.001 0.001; visual mesh filename=package://concert_resources/models/modular/meshes/concert/c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 scale=0.001 0.001 0.001
- added link J4_E_stator, mass 3.3057881; collision mesh filename=package://concert_resources/models/modular/meshes/concert/s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 scale=0.001 0.001 0.001; visual mesh filename=package://concert_resources/models/modular/meshes/concert/c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 scale=0.001 0.001 0.001
- added link J5_E_stator, mass 3.2592751; collision mesh filename=package://concert_resources/models/modular/meshes/concert/s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 scale=0.001 0.001 0.001; visual mesh filename=package://concert_resources/models/modular/meshes/concert/c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 scale=0.001 0.001 0.001
- added link L_1_E, mass 0.57797267; collision mesh filename=package://concert_resources/models/modular/meshes/concert/s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 scale=0.001 0.001 0.001; visual mesh filename=package://concert_resources/models/modular/meshes/concert/c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 scale=0.001 0.001 0.001
- added link L_2_E, mass 1.1481338; collision mesh filename=package://concert_resources/models/modular/meshes/concert/s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 scale=0.001 0.001 0.001; visual mesh filename=package://concert_resources/models/modular/meshes/concert/c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 scale=0.001 0.001 0.001
- added link L_3_E, mass 0.56725368; collision mesh filename=package://concert_resources/models/modular/meshes/concert/s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 scale=0.001 0.001 0.001; visual mesh filename=package://concert_resources/models/modular/meshes/concert/c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 scale=0.001 0.001 0.001
- added link L_4_E, mass 1.1588784; collision mesh filename=package://concert_resources/models/modular/meshes/concert/s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 scale=0.001 0.001 0.001; visual mesh filename=package://concert_resources/models/modular/meshes/concert/c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 scale=0.001 0.001 0.001
- added link L_5_E, mass 0.56725368; collision mesh filename=package://concert_resources/models/modular/meshes/concert/s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 scale=0.001 0.001 0.001; visual mesh filename=package://concert_resources/models/modular/meshes/concert/c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 scale=0.001 0.001 0.001
- added link ee_E, mass 1.305; collision cylinder length=0.2 radius=0.02; visual cylinder length=0.2 radius=0.02
Joints:
- added joint J1_E: type revolute, parent J1_E_stator, child L_1_E, origin xyz=0.0 0.0 0.22316 rpy=0.0 -0.0 0.0, axis 0 0 1, limit lower=-3.0 upper=3.0 effort=460.0 velocity=1.77
- added joint J2_E: type revolute, parent J2_E_stator, child L_2_E, origin xyz=0.0 0.13666 0.0875 rpy=-1.5707963267948966 -0.0 0.0, axis 0 0 1, limit lower=-3.0 upper=3.0 effort=460.0 velocity=1.77
- added joint J3_E: type revolute, parent J3_E_stator, child L_3_E, origin xyz=0.0 0.0 0.22316 rpy=0.0 -0.0 0.0, axis 0 0 1, limit lower=-3.0 upper=3.0 effort=314.0 velocity=2.36
- added joint J4_E: type revolute, parent J4_E_stator, child L_4_E, origin xyz=0.0 0.13666 0.0875 rpy=-1.5707963267948966 -0.0 0.0, axis 0 0 1, limit lower=-3.0 upper=3.0 effort=314.0 velocity=2.36
- added joint J5_E: type revolute, parent J5_E_stator, child L_5_E, origin xyz=0.0 0.0 0.22316 rpy=0.0 -0.0 0.0, axis 0 0 1, limit lower=-3.0 upper=3.0 effort=314.0 velocity=2.36
- added joint L_5_fixed_joint_1_E: type fixed, parent L_5_E, child ee_E, origin xyz=0.0 0.0 0.22184 rpy=0.0 -0.0 0.0, axis 0 0 1
- added joint fixed_J1_E: type fixed, parent mobile_base, child J1_E_stator, origin xyz=0.2 0.0 0.016 rpy=0.0 -0.0 3.141592653589793, axis 0 0 1
- added joint fixed_J2_E: type fixed, parent L_1_E, child J2_E_stator, origin xyz=0.0 0.0 0.02184 rpy=0.0 -0.0 0.0, axis 0 0 1
- added joint fixed_J3_E: type fixed, parent L_2_E, child J3_E_stator, origin xyz=0.0 -0.0875 0.0195 rpy=-1.5707963267948966 -0.0 3.141592653589793, axis 0 0 1
- added joint fixed_J4_E: type fixed, parent L_3_E, child J4_E_stator, origin xyz=0.0 0.0 0.02184 rpy=0.0 -0.0 0.0, axis 0 0 1
- added joint fixed_J5_E: type fixed, parent L_4_E, child J5_E_stator, origin xyz=0.0 -0.0875 0.0195 rpy=-1.5707963267948966 -0.0 3.141592653589793, axis 0 0 1
